Commit message: Week 2 Day 2: Add wheels, caster, and sensor mount to URDF

File: ros2_ws/src/my_robot_description/urdf/my_robot.urdf (robot description, URDF)
Before this commit: robot my_robot, 1 links, 0 joints
Links:
- added link caster_wheel_link; visual sphere radius=0.025
- added link left_wheel_link; visual cylinder length=0.03 radius=0.05
- added link right_wheel_link; visual cylinder length=0.03 radius=0.05
- added link sensor_mount_link; visual box size=0.05 0.05 0.05
Joints:
- added joint caster_wheel_joint: type fixed, parent base_link, child caster_wheel_link, origin xyz=0.15 0 0.025 rpy=0 0 0
- added joint left_wheel_joint: type continuous, parent base_link, child left_wheel_link, origin xyz=0 0.165 0.05 rpy=0 0 0, axis 0 1 0
- added joint right_wheel_joint: type continuous, parent base_link, child right_wheel_link, origin xyz=0 -0.165 0.05 rpy=0 0 0, axis 0 1 0
- added joint sensor_mount_joint: type fixed, parent base_link, child sensor_mount_link, origin xyz=0 0 0.15 rpy=0 0 0
